File: BD/BD.kicad_pcb (KiCad board)
At the start: 2 copper layers, 100 x 100 mm, 57 parts, among them P1 bateria 7.4 V, P2 HC-06 (BT), P3 SILNIK1, P4 Modol startujacy, P5 PROGRAMAT, P7 SILNIK2, SW1 SWITCH_INV, SW2 SW_PUSH, U1 LM1117, U10 TB6612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

Commit message: footprinty zrobione
Parts:
- C1, C13, C2, C3, C4: footprint Capacitors_SMD:C_0201 -> Capacitors_SMD:C_0402
- C10, C11, C12: footprint Capacitors_SMD:C_0201 -> Capacitors_SMD:C_0603
- C14, C16, C18, C19, C22, C9: footprint Capacitors_SMD:C_0201 -> Capacitors_SMD:C_0805
- C15, C17, C20, C21, C5, C6, C7, C8: footprint Capacitors_SMD:c_elec_3x5.3 -> Capacitors_Tantalum_SMD:TantalC_SizeR_EIA-2012
- D1, DB1, DN1: footprint LEDs:LED-3MM -> LEDs:LED-5MM
- P1, P3, P7: footprint Pin_Headers:Pin_Header_Angled_1x02 -> Socket_Strips:Socket_Strip_Straight_1x02
- P2, P5: footprint misc W:Pin_Header_Straight_1x04 -> Socket_Strips:Socket_Strip_Straight_1x04
- P4: footprint Pin_Headers:Pin_Header_Angled_1x03 -> Socket_Strips:Socket_Strip_Straight_1x03
- R1, R11, R12, R2, R3, R4, R5, R6: footprint Resistors_SMD:R_0201 -> Resistors_SMD:R_0805
- R10, R7, R8, R9: footprint Resistors_SMD:R_0201 -> Resistors_SMD:R_0603
- SP1: footprint Air_Coils_SML_NEOSID:Neosid_Air-Coil_SML_1turn_HDM0131A -> Buzzer_moj
- SW1: value SWITCH_INV -> SPST; footprint Buttons_Switches_SMD:SW_SPDT_PCM12 -> Buttons_Switches_ThroughHole:SW_DIP_x1_Slide
- SW2: footprint Air_Coils_SML_NEOSID:Neosid_Air-Coil_SML_1turn_HDM0131A -> Buttons_Switches_ThroughHole:SW_PUSH_6mm
- U9: footprint misc W:LQFP48 -> STM:STM32F051C8T6
- moved U4 180.0 mm to (92.4, 109.6)
- moved P1 165.6 mm to (107.5, 135.0)
- moved C2 152.8 mm to (165.0, 110.0)
- moved C3 151.4 mm to (129.4, 100.0)
- moved R8 150.2 mm to (120.0, 125.0)
- moved U2 149.2 mm to (197.4, 74.6)
- moved U8 147.6 mm to (148.5, 110.0)
- moved R2 145.8 mm to (160.0, 130.0)
- moved R6 135.4 mm to (130.0, 130.0), turned to 0 degrees
- moved C5 131.5 mm to (130.0, 105.0), turned to 0 degrees
- moved R1 131.4 mm to (170.9, 130.0)
- moved R3 128.6 mm to (155.0, 130.0)
- moved U7 121.7 mm to (155.0, 110.0)
- moved U6 117.9 mm to (133.1, 65.0), turned to 0 degrees
- moved C1 117.4 mm to (164.4, 100.0)
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Connections:
- SW1 pad 1: VCC -> Net-(P1-Pad2)
- SW1 pad 2: Net-(P1-Pad2) -> VCC
Routing:
- net GND: track 0.55 -> 0.00 mm
Other:
- board outline removed

Commit message: plytka_pcb
Parts:
- U2, U3, U4, U5: moved to B.Cu
- moved U4 98.7 mm to (190.8, 101.6), turned to 90 degrees
- moved SP1 95.3 mm to (189.7, 114.1), turned to 270 degrees
- moved R8 79.5 mm to (189.5, 86.4)
- moved U2 76.5 mm to (121.4, 84.2), turned to 180 degrees
- moved SW2 70.0 mm to (126.7, 116.8), turned to 90 degrees
- moved C15 69.9 mm to (139.5, 144.9), turned to 90 degrees
- moved C16 67.7 mm to (134.4, 144.9), turned to 270 degrees
- moved R11 67.6 mm to (168.2, 113.8), turned to 180 degrees
- moved D1 66.3 mm to (131.3, 99.5)
- moved C20 65.3 mm to (152.2, 144.8), turned to 90 degrees
- moved P2 65.0 mm to (112.9, 116.6), turned to 180 degrees
- moved C21 60.1 mm to (155.4, 144.8), turned to 90 degrees
- moved C17 59.4 mm to (142.9, 144.9), turned to 90 degrees
- moved R1 59.3 mm to (122.6, 95.7)
- moved U1 58.0 mm to (148.9, 81.9), turned to 90 degrees
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Connections:
- U9 pad 10: SHARP1 -> S2/IN1
- U9 pad 11: KTIR1 -> S2/IN2
- U9 pad 12: SHARP2 -> S2/PWM
- U9 pad 13: SHARP3 -> S1/PWM
- U9 pad 14: KTIR2 -> S1/IN2
- U9 pad 15: SHARP4 -> S1/IN1
- U9 pad 25: S1/IN1 -> SHARP1
- U9 pad 26: S1/IN2 -> KTIR1
- U9 pad 27: S1/PWM -> SHARP2
- U9 pad 28: S2/PWM -> SHARP3
- U9 pad 29: Net-(U9-Pad29) -> KTIR2
- U9 pad 30: S2/IN1 -> SHARP4
- U9 pad 31: S2/IN2 -> Net-(U9-Pad31)
Routing:
- net KTIR2: track 0.00 -> 5.70 mm
- net Net-(R9-Pad1): track 0.00 -> 2.69 mm
- net +3V3: track 0.00 -> 1.38 mm
Other:
- board outline added: 95 x 70 mm

Commit message: można szyczyć?
Parts:
- P3, P7, R10, R7, R8, R9, U7, U8: moved to B.Cu
- U2, U3, U4, U5: moved to F.Cu
- moved D1 46.7 mm to (177.6, 105.8), turned to 180 degrees
- moved C19 33.4 mm to (127.5, 139.3)
- moved C18 32.2 mm to (167.6, 135.4)
- moved R6 30.9 mm to (168.4, 105.6), turned to 180 degrees
- moved C17 29.3 mm to (170.4, 135.1)
- moved C20 28.4 mm to (124.4, 139.6)
- moved C12 27.4 mm to (139.0, 114.5), turned to 90 degrees
- moved C13 25.9 mm to (146.3, 118.2), turned to 180 degrees
- moved C11 23.6 mm to (140.7, 114.5), turned to 90 degrees
- moved C14 21.2 mm to (146.3, 120.2), turned to 180 degrees
- moved C15 18.3 mm to (124.3, 134.6), turned to 270 degrees
- moved SW1 18.0 mm to (138.2, 99.9), turned to 270 degrees
- moved C21 15.9 mm to (170.5, 139.9), turned to 270 degrees
- moved P4 13.6 mm to (167.6, 122.5), turned to 180 degrees
- moved U12 13.3 mm to (135.1, 135.1), turned to 180 degrees
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Routing:
- net KTIR2: track 5.70 -> 0.00 mm
- net Net-(R9-Pad1): track 2.69 -> 0.00 mm
- net +3V3: track 1.38 -> 0.00 mm
Other:
- net class Default: via_dia 1 -> 1.3; via_drill 0.6 -> 0.5
- rule via_min_drill: 0.6 -> 0.5
- rule via_min_size: 1 -> 1.2

Commit message: moze zadziala?
Parts:
- moved P5 12.7 mm to (111.3, 116.2), turned to 180 degrees
- moved P2 9.55 mm to (118.7, 124.2), turned to 90 degrees
- moved C9 8.23 mm to (139.4, 122.0), turned to 90 degrees
- moved P4 7.26 mm to (164.0, 116.2)
- moved SW2 5.20 mm to (129.1, 113.0), turned to 0 degrees
- moved P1 2.21 mm to (137.8, 90.6)
- moved C10 1.29 mm to (155.0, 107.6)
- moved C21 1.16 mm to (170.6, 138.7)
- moved C15 0.93 mm to (124.2, 133.7), turned to 90 degrees
- moved C17 0.77 mm to (170.5, 134.3)
- moved C20 0.75 mm to (124.3, 138.8), turned to 270 degrees
- moved SW1 0.53 mm to (137.9, 99.5)
- moved C22 0.47 mm to (167.6, 139.1)
- moved C19 0.21 mm to (127.5, 139.1), turned to 270 degrees
- turned C16 to 270 degrees
Routing:
- net +3V3: track 0.00 -> 417.7 mm, vias 0 -> 5
- net +5V: track 0.00 -> 214.6 mm, vias 0 -> 5
- net GND: track 0.00 -> 111.1 mm
- net VCC: track 0.00 -> 108.5 mm, vias 0 -> 1
- net KTIR2: track 0.00 -> 60.6 mm, vias 0 -> 1
- net SHARP4: track 0.00 -> 57.4 mm
- net KTIR1: track 0.00 -> 56.5 mm, vias 0 -> 1
- net SHARP1: track 0.00 -> 46.8 mm
- net PROG1: track 0.00 -> 44.5 mm, vias 0 -> 1
- net SHARP3: track 0.00 -> 44.4 mm
- net S2/PWM: track 0.00 -> 40.7 mm
- net S2/IN2: track 0.00 -> 39.7 mm
- net SHARP2: track 0.00 -> 39.2 mm
- net S2/IN1: track 0.00 -> 38.8 mm
- net PROG2: track 0.00 -> 37.7 mm, vias 0 -> 1
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Other:
- outline, holes or cut-outs redrawn
- net class Default: clearance 0.254 -> 0.2
- rule trace_clearance: 0.254 -> 0.2

Commit message: koniec?
Routing:
- net Net-(R7-Pad1): track 5.64 -> 14.6 mm
- net GND: track 111.1 -> 116.8 mm, vias 0 -> 2
- net (no net): track 0.00 -> 1.66 mm, vias 0 -> 3
- added copper zone on B.Cu, net GND
- added copper zone on F.Cu, net GND
Changed lines of the file:
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@@
   (general
     (links 166)
-    (no_connects 38)
+    (no_connects 17)
     (area 97.2375 77.3275 197.7525 150.075001)
     (thickness 1.6)
     (drawings 43)
-    (tracks 590)
+    (tracks 611)
     (zones 0)
     (modules 57)
@@
     (pad_to_mask_clearance 0.2)
     (aux_axis_origin 76.02 164.95)
+    (grid_origin 189.34 83.26)
     (visible_elements 7FFFFFFF)
     (pcbplotparams
@@
   (gr_line (start 140.99 129.01) (end 115.01 129.01) (layer Dwgs.User) (width 0.2))
   (gr_line (start 140.99 141) (end 140.99 129.01) (layer Dwgs.User) (width 0.2))
-  (target plus (at 127.160328 100.595397) (size 5) (width 0.15) (layer Edge.Cuts))
-  (target plus (at 168.687574 98.921426) (size 5) (width 0.15) (layer Edge.Cuts))
+  (target plus (at 127.121862 99.199841) (size 5) (width 0.15) (layer Edge.Cuts))
+  (target plus (at 167.982785 99.161052) (size 5) (width 0.15) (layer Edge.Cuts))
   (gr_line (start 180 150) (end 165 150) (layer Edge.Cuts) (width 0.15))
   (gr_line (start 180 120) (end 180 150) (layer Edge.Cuts) (width 0.15))
@@
   (gr_line (start 165 150) (end 115 150) (layer Edge.Cuts) (width 0.15))
   (gr_line (start 100 80) (end 180 80) (layer Edge.Cuts) (width 0.15))
+  (segment (start 132.38 114.79) (end 132.35 114.79) (width 0.254) (layer F.Cu) (net 0))
+  (segment (start 132.35 114.79) (end 132.32 114.82) (width 0.254) (layer F.Cu) (net 0))
+  (via (at 132.32 114.82) (size 1.3) (drill 0.5) (layers F.Cu B.Cu) (net 0))
+  (segment (start 131.83 83.21) (end 132.64 83.21) (width 0.3356) (layer B.Cu) (net 0))
+  (via (at 132.64 83.21) (size 1.3) (drill 0.5) (layers F.Cu B.Cu) (net 0))
+  (segment (start 129.39 137.29) (end 129.02 137.66) (width 0.3048) (layer B.Cu) (net 0))
+  (segment (start 129.19 137.42) (end 129.26 137.42) (width 0.3048) (layer F.Cu) (net 0))
+  (segment (start 129.26 137.42) (end 129.39 137.29) (width 0.3048) (layer F.Cu) (net 0))
+  (via (at 129.39 137.29) (size 1.3) (drill 0.5) (layers F.Cu B.Cu) (net 0))
+  (segment (start 189.435 83.295) (end 186.155 83.295) (width 0.889) (layer B.Cu) (net 1))
+  (segment (start 186.155 83.295) (end 186.09 83.23) (width 0.889) (layer B.Cu) (net 1))
+  (via (at 186.09 83.23) (size 1.3) (drill 0.5) (layers F.Cu B.Cu) (net 1))
+  (segment (start 165.72 137.42) (end 166.369999 138.069999) (width 0.3048) (layer B.Cu) (net 1))
+  (segment (start 166.369999 138.069999) (end 166.589999 138.069999) (width 0.3048) (layer B.Cu) (net 1))
+  (segment (start 165.79 136.2052) (end 166.11 136.5252) (width 0.3048) (layer F.Cu) (net 1))
+  (segment (start 164.9198 135.335) (end 165.79 136.2052) (width 0.3048) (layer F.Cu) (net 1))
+  (segment (start 165.79 136.2052) (end 165.79 137.35) (width 0.3048) (layer F.Cu) (net 1))
+  (segment (start 165.79 137.35) (end 165.72 137.42) (width 0.3048) (layer F.Cu) (net 1))
+  (via (at 165.72 137.42) (size 1.3) (drill 0.5) (layers F.Cu B.Cu) (net 1))
   (segment (start 177.44 121.67) (end 177.44 120.3652) (width 0.3048) (layer F.Cu) (net 1))
   (segment (start 177.44 120.3652) (end 177.44 113.77) (width 0.3048) (layer F.Cu) (net 1))
@@
   (segment (start 166.2352 136.4) (end 167.55 136.4) (width 0.3048) (layer F.Cu) (net 1))
   (segment (start 163.74 135.335) (end 164.9198 135.335) (width 0.3048) (layer F.Cu) (net 1))
-  (segment (start 164.9198 135.335) (end 166.11 136.5252) (width 0.3048) (layer F.Cu) (net 1))
   (segment (start 152.808548 95.02183) (end 152.808548 97.19226) (width 1.27) (layer F.Cu) (net 1))
   (segment (start 152.808548 97.19226) (end 152.72 97.280808) (width 1.27) (layer F.Cu) (net 1))
@@
   (segment (start 145.484568 87.74183) (end 145.484568 91.54581) (width 0.889) (layer F.Cu) (net 7))
   (segment (start 145.484568 91.54581) (end 145.510588 91.57183) (width 0.889) (layer F.Cu) (net 7))
+  (segment (start 191.86 86.29) (end 191.2 86.29) (width 0.3048) (layer B.Cu) (net 8))
+  (segment (start 124.24 132.51) (end 126.8548 132.51) (width 0.3048) (layer F.Cu) (net 8))
+  (segment (start 126.8548 132.51) (end 127.5 133.1552) (width 0.3048) (layer F.Cu) (net 8))
+  (segment (start 127.5 133.1552) (end 127.5 133.96) (width 0.3048) (layer F.Cu) (net 8))
   (segment (start 127.5 133.96) (end 127.856091 133.96) (width 0.3048) (layer F.Cu) (net 8))
   (segment (start 127.856091 133.96) (end 129.341091 135.445) (width 0.3048) (layer F.Cu) (net 8))
   (segment (start 130.3302 135.445) (end 131.51 135.445) (width 0.3048) (layer F.Cu) (net 8))
   (segment (start 129.341091 135.445) (end 130.3302 135.445) (width 0.3048) (layer F.Cu) (net 8))
-  (segment (start 124.24 132.51) (end 126.8548 132.51) (width 0.3048) (layer F.Cu) (net 8))
-  (segment (start 126.8548 132.51) (end 127.5 133.1552) (width 0.3048) (layer F.Cu) (net 8))
-  (segment (start 127.5 133.1552) (end 127.5 133.96) (width 0.3048) (layer F.Cu) (net 8))
   (segment (start 122.45057 132.3) (end 122.45057 131.464198) (width 0.889) (layer F.Cu) (net 8))
   (segment (start 122.45057 136.52574) (end 122.45057 132.3) (width 0.889) (layer F.Cu) (net 8))
@@
   (segment (start 156.705499 87.314501) (end 104.864501 87.314501) (width 0.889) (layer B.Cu) (net 8))
   (segment (start 104.864501 87.314501) (end 103.74 86.19) (width 0.889) (layer B.Cu) (net 8))
-  (segment (start 191.86 86.29) (end 191.2 86.29) (width 0.3048) (layer B.Cu) (net 8))
   (segment (start 191.2 86.29) (end 190.43 86.29) (width 0.3048) (layer B.Cu) (net 8))
   (segment (start 162.49 81.53) (end 162.49 82.449238) (width 0.889) (layer B.Cu) (net 8))
@@
   (segment (start 165.27 110.28) (end 167.61 112.62) (width 0.254) (layer F.Cu) (net 27))
   (segment (start 167.61 112.62) (end 167.61 112.92) (width 0.254) (layer F.Cu) (net 27))
+  (segment (start 183.89 82.3) (end 184.695 81.495) (width 0.3048) (layer B.Cu) (net 28))
+  (segment (start 184.695 81.495) (end 189.435 81.495) (width 0.3048) (layer B.Cu) (net 28))
+  (segment (start 183.89 84.48) (end 183.89 82.3) (width 0.3048) (layer B.Cu) (net 28))
+  (segment (start 184.507799 85.097799) (end 183.89 84.48) (width 0.3048) (layer B.Cu) (net 28))
+  (segment (start 188.432599 85.097799) (end 184.507799 85.097799) (width 0.3048) (layer B.Cu) (net 28))
   (segment (start 188.9 86.32) (end 188.9 85.5652) (width 0.3048) (layer B.Cu) (net 28))
-  (segment (start 188.432599 82.147401) (end 189.085 81.495) (width 0.3048) (layer B.Cu) (net 28))
   (segment (start 188.9 85.5652) (end 188.432599 85.097799) (width 0.3048) (layer B.Cu) (net 28))
-  (segment (start 188.432599 85.097799) (end 188.432599 82.147401) (width 0.3048) (layer B.Cu) (net 28))
   (segment (start 189.085 81.495) (end 189.435 81.495) (width 0.3048) (layer B.Cu) (net 28))
   (segment (start 190.27 89.48) (end 187.479499 92.270501) (width 0.254) (layer F.Cu) (net 29))
@@
   (segment (start 131.412001 133.397001) (end 131.51 133.495) (width 0.254) (layer F.Cu) (net 53))
   (segment (start 149.64 115.78) (end 149.64 120.82) (width 0.254) (layer F.Cu) (net 53))
+  (zone (net 1) (net_name GND) (layer F.Cu) (hatch edge 0.508)
+    (connect_pads (clearance 0.508))
+    (min_thickness 0.254)
+    (fill yes (arc_segments 16) (thermal_gap 0.508) (thermal_bridge_width 0.508))
+    (polygon
+      (pts
+        (xy 100.01 79.99) (xy 194.99 80.01) (xy 194.97 119.99) (xy 180.01 120) (xy 179.97 150)
+        (xy 115 149.98) (xy 114.98 120.01) (xy 100 120)
+      )
+    )
+  )
+  (zone (net 1) (net_name GND) (layer B.Cu) (hatch edge 0.508)
+    (connect_pads (clearance 0.508))
+    (min_thickness 0.254)
+    (fill yes (arc_segments 16) (thermal_gap 0.508) (thermal_bridge_width 0.508))
+    (polygon
+      (pts
+        (xy 100 80.01) (xy 100 120) (xy 114.99 120.02) (xy 115 150) (xy 179.99 149.98)
+        (xy 180.02 120.01) (xy 194.98 120) (xy 194.98 80.02) (xy 100 80.02) (xy 100 80.02)
+      )
+    )
+  )
 )

Commit message: hmm
Routing:
- net VCC: track 108.5 -> 129.7 mm, vias 1 -> 2
- net GND: track 116.8 -> 111.1 mm, vias 2 -> 0
- net +3V3: track 417.7 -> 420.1 mm
- net S1/IN2: track 33.2 -> 34.9 mm
- net (no net): track 1.66 -> 0.07 mm, vias 3 -> 1
- net S1/IN1: track 33.0 -> 33.8 mm
- net S1/PWM: track 33.1 -> 33.8 mm
- removed copper zone on B.Cu, net GND
- removed copper zone on F.Cu, net GND

Commit message: dsf
Routing:
- net (no net): track 0.07 -> 14.8 mm, vias 1 -> 4
- added copper zone on B.Cu, net GND
- added copper zone on F.Cu, net GND
Changed lines of the file:
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@@
   (general
     (links 166)
-    (no_connects 17)
+    (no_connects 37)
     (area 97.2375 77.3275 197.7525 150.075001)
     (thickness 1.6)
     (drawings 43)
-    (tracks 621)
+    (tracks 655)
     (zones 0)
     (modules 57)
@@
   )
   (setup
-    (last_trace_width 0.889)
+    (last_trace_width 1.27)
     (user_trace_width 0.254)
     (user_trace_width 0.3048)
@@
   (gr_line (start 165 150) (end 115 150) (layer Edge.Cuts) (width 0.15))
   (gr_line (start 100 80) (end 180 80) (layer Edge.Cuts) (width 0.15))
-  (segment (start 132.38 114.79) (end 132.35 114.79) (width 0.254) (layer F.Cu) (net 0))
-  (segment (start 132.35 114.79) (end 132.32 114.82) (width 0.254) (layer F.Cu) (net 0))
-  (via (at 132.32 114.82) (size 1.3) (drill 0.5) (layers F.Cu B.Cu) (net 0))
+  (segment (start 131.83 115.5) (end 132.78 115.5) (width 1.27) (layer B.Cu) (net 0))
+  (segment (start 131.33 115) (end 131.83 115.5) (width 1.27) (layer B.Cu) (net 0))
+  (segment (start 131.33 114.94) (end 131.33 115) (width 1.27) (layer B.Cu) (net 0))
+  (segment (start 131.39 114.88) (end 131.33 114.94) (width 1.27) (layer B.Cu) (net 0))
+  (segment (start 131.39 114.6) (end 131.39 114.88) (width 1.27) (layer B.Cu) (net 0))
+  (segment (start 131.79 114.2) (end 131.39 114.6) (width 1.27) (layer B.Cu) (net 0))
+  (segment (start 132.48 114.2) (end 131.79 114.2) (width 1.27) (layer B.Cu) (net 0))
+  (segment (start 133.049238 114.769238) (end 132.48 114.2) (width 1.27) (layer B.Cu) (net 0))
+  (segment (start 133.049238 115) (end 133.049238 114.769238) (width 1.27) (layer B.Cu) (net 0))
+  (segment (start 131.79 115.34) (end 132.709238 115.34) (width 1.27) (layer B.Cu) (net 0))
+  (segment (start 132.709238 115.34) (end 133.049238 115) (width 1.27) (layer B.Cu) (net 0))
+  (segment (start 132.47 115.62) (end 132.07 115.62) (width 1.27) (layer F.Cu) (net 0))
+  (via (at 131.79 115.34) (size 1.3) (drill 0.5) (layers F.Cu B.Cu) (net 0))
+  (segment (start 132.07 115.62) (end 131.79 115.34) (width 1.27) (layer F.Cu) (net 0))
+  (segment (start 132.67 115.42) (end 132.47 115.62) (width 1.27) (layer F.Cu) (net 0))
+  (segment (start 132.67 115.19) (end 132.67 115.42) (width 1.27) (layer F.Cu) (net 0))
+  (segment (start 132.88 114.98) (end 132.67 115.19) (width 1.27) (layer F.Cu) (net 0))
+  (segment (start 132.88 114.35) (end 132.88 114.98) (width 1.27) (layer F.Cu) (net 0))
+  (segment (start 132.61141 114.08141) (end 132.88 114.35) (width 1.27) (layer F.Cu) (net 0))
+  (segment (start 132.07859 114.08141) (end 132.61141 114.08141) (width 1.27) (layer F.Cu) (net 0))
+  (segment (start 131.38 114.78) (end 132.07859 114.08141) (width 1.27) (layer F.Cu) (net 0))
+  (segment (start 131.31 114.78) (end 131.38 114.78) (width 1.27) (layer F.Cu) (net 0))
+  (segment (start 129.39 137.24) (end 130.039999 137.889999) (width 0.254) (layer B.Cu) (net 0))
+  (segment (start 130.039999 137.889999) (end 130.039999 138.279999) (width 0.254) (layer B.Cu) (net 0))
+  (segment (start 129.3 137.87) (end 129.3 137.33) (width 0.254) (layer F.Cu) (net 0))
+  (segment (start 129.3 137.33) (end 129.39 137.24) (width 0.254) (layer F.Cu) (net 0))
+  (via (at 129.39 137.24) (size 1.3) (drill 0.5) (layers F.Cu B.Cu) (net 0))
+  (segment (start 165.81 138.22) (end 164.890762 138.22) (width 0.254) (layer B.Cu) (net 0))
+  (segment (start 164.890762 138.22) (end 164.550762 138.56) (width 0.254) (layer B.Cu) (net 0))
+  (segment (start 165.73 138.19) (end 165.78 138.19) (width 0.254) (layer F.Cu) (net 0))
+  (segment (start 165.78 138.19) (end 165.81 138.22) (width 0.254) (layer F.Cu) (net 0))
+  (via (at 165.81 138.22) (size 1.3) (drill 0.5) (layers F.Cu B.Cu) (net 0))
+  (segment (start 186.63 83.32) (end 185.93 83.32) (width 0.254) (layer F.Cu) (net 0))
+  (segment (start 186.72 83.23) (end 186.63 83.32) (width 0.254) (layer F.Cu) (net 0))
+  (segment (start 187.27 83.24) (end 186.73 83.24) (width 0.254) (layer B.Cu) (net 0))
+  (segment (start 186.73 83.24) (end 186.72 83.23) (width 0.254) (layer B.Cu) (net 0))
+  (via (at 186.72 83.23) (size 1.3) (drill 0.5) (layers F.Cu B.Cu) (net 0))
   (segment (start 165.79 136.2052) (end 166.11 136.5252) (width 0.3048) (layer F.Cu) (net 1))
   (segment (start 164.9198 135.335) (end 165.79 136.2052) (width 0.3048) (layer F.Cu) (net 1))
@@
   (segment (start 131.412001 133.397001) (end 131.51 133.495) (width 0.254) (layer F.Cu) (net 53))
   (segment (start 149.64 115.78) (end 149.64 120.82) (width 0.254) (layer F.Cu) (net 53))
+  (zone (net 1) (net_name GND) (layer F.Cu) (hatch edge 0.508)
+    (connect_pads (clearance 0.508))
+    (min_thickness 0.254)
+    (fill yes (arc_segments 16) (thermal_gap 0.508) (thermal_bridge_width 0.508))
+    (polygon
+      (pts
+        (xy 100.01 80) (xy 100.01 119.98) (xy 114.98 120.02) (xy 115.01 149.97) (xy 179.98 149.97)
+        (xy 180 120) (xy 194.98 119.96) (xy 194.98 80)
+      )
+    )
+  )
+  (zone (net 1) (net_name GND) (layer B.Cu) (hatch edge 0.508)
+    (connect_pads (clearance 0.508))
+    (min_thickness 0.254)
+    (fill yes (arc_segments 16) (thermal_gap 0.508) (thermal_bridge_width 0.508))
+    (polygon
+      (pts
+        (xy 100.02 80.02) (xy 194.98 80) (xy 194.99 119.95) (xy 179.99 120.04) (xy 179.97 150.01)
+        (xy 115 149.97) (xy 114.98 120.02) (xy 100 119.98) (xy 100.01 80.02)
+      )
+    )
+  )
 )

Commit message: yep
Parts:
- R11, R5, R6: moved to B.Cu
Routing:
- net +5V: track 214.6 -> 179.6 mm, vias 5 -> 7
- net SHARP4: track 57.4 -> 43.7 mm
- net Net-(R12-Pad1): track 33.3 -> 20.3 mm, vias 0 -> 1
- net (no net): track 14.8 -> 3.69 mm, vias 4 -> 5
- net SHARP3: track 44.4 -> 52.7 mm
- net GND: track 111.1 -> 103.2 mm
- net SHARP1: track 46.8 -> 40.6 mm
- net Net-(P3-Pad2): track 6.88 -> 12.6 mm, vias 0 -> 1
- net Net-(P7-Pad2): track 6.67 -> 11.2 mm, vias 0 -> 1
- net VCC: track 129.7 -> 132.8 mm
- net Net-(P3-Pad1): track 16.0 -> 17.4 mm, vias 0 -> 1
- net Net-(P7-Pad1): track 14.8 -> 15.4 mm, vias 0 -> 1
- net +3V3: track 420.1 -> 419.5 mm
- net LED1: track 15.9 -> 16.3 mm, vias 0 -> 1
- net LED2: vias 0 -> 1
Other:
- board text added: "5 przelotek uziemien"
