File: BD/BD.kicad_pcb (KiCad board)
At the start: 2 copper layers, 95 x 70 mm, 57 parts, among them P1 bateria 7.4 V, P2 HC-06 (BT), P3 SILNIK1, P4 Modol startujacy, P5 PROGRAMAT, P7 SILNIK2, SW1 SPST, SW2 SW_PUSH, U1 LM1117, U10 TB6612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

Commit message: tak?
Parts:
- moved P3 0.34 mm to (151.5, 136.0)
- moved P7 0.13 mm to (143.3, 136.1)
Routing:
- net GND: track 103.2 -> 110.3 mm, vias 0 -> 2
- net Net-(R7-Pad1): track 14.6 -> 9.11 mm, vias 0 -> 2
- net PROG1: track 44.5 -> 49.7 mm
- net PROG2: track 37.7 -> 39.5 mm
- net (no net): track 3.69 -> 5.46 mm, vias 5 -> 2

Commit message: Zwiekszenie plytki
Parts:
- moved R7 19.4 mm to (188.2, 67.0)
- moved R8 19.3 mm to (192.2, 67.0)
- moved R10 19.2 mm to (105.8, 67.0)
- moved R9 19.2 mm to (102.8, 67.0)
- moved U7 18.3 mm to (191.0, 64.1)
- moved U8 18.3 mm to (104.5, 64.1)
- moved R1 14.8 mm to (126.0, 80.0)
- moved R4 14.8 mm to (177.6, 79.8)
- moved C4 14.7 mm to (173.1, 79.8)
- moved C1 14.7 mm to (121.0, 80.0)
- moved U2 14.4 mm to (124.0, 70.0)
- moved U5 14.2 mm to (176.0, 70.0)
Routing:
- net +3V3: track 419.5 -> 458.2 mm
- net +5V: track 179.6 -> 204.2 mm
- net KTIR1: track 56.5 -> 74.6 mm
- net SHARP2: track 39.5 -> 52.6 mm
- net KTIR2: track 60.6 -> 72.5 mm
- net SHARP3: track 52.7 -> 56.4 mm
- net Net-(R4-Pad1): track 6.29 -> 4.83 mm
- net Net-(R9-Pad1): track 6.15 -> 4.84 mm
- net Net-(R7-Pad1): track 9.11 -> 7.81 mm, vias 2 -> 0
- net Net-(C1-Pad2): track 6.27 -> 5.49 mm
- net GND: track 110.3 -> 109.6 mm, vias 2 -> 1
- net (no net): track 5.46 -> 4.81 mm, vias 2 -> 1
Other:
- board size 95 x 70 mm -> 95 x 90 mm

Commit message: Inventor wersja 1
Parts:
- moved C4 11.3 mm to (168.1, 90.0)
- moved R4 10.8 mm to (174.1, 90.0)
- moved U5 10.4 mm to (172.5, 79.8)
- moved C1 10.0 mm to (120.0, 90.0)
- moved R1 10.0 mm to (126.0, 90.0)
- moved U2 10.0 mm to (124.0, 80.0)
Routing:
- net +5V: track 204.2 -> 188.7 mm
- net SHARP2: track 52.6 -> 41.2 mm
- net (no net): track 4.81 -> 7.97 mm
- net Net-(R7-Pad1): track 7.81 -> 4.66 mm
- net GND: track 109.6 -> 111.9 mm
- net SHARP3: track 56.4 -> 54.3 mm
- removed copper zone on F.Cu, net GND

Commit message: moze
Routing:
- net GND: track 111.9 -> 145.5 mm, vias 1 -> 2
- net (no net): track 7.97 -> 13.9 mm, vias 1 -> 5
- net SHARP3: track 54.3 -> 49.4 mm
- net Net-(P3-Pad1): track 17.4 -> 22.3 mm
- net Net-(P7-Pad1): track 15.4 -> 19.6 mm
- added copper zone on F.Cu, net GND
