File: BD/BD.sch (KiCad schematic (older format))
At the start: 45 parts, among them P1 CONN_01X02, P2 SILNIK1, P3 SILNIK2, SW1 SWITCH_INV, SW2 SW_PUSH, U1 LM1117, U10 L293D, U2 SHARP_40CM, U3 SHARP_40CM, U4 SHARP_40CM, U5 SHARP_40CM, U6 LM1117, U7 KTIR0711S, U8 KTIR0711S, U9 STM32F051C8Tx

Commit message: pierwsze zmiany
Parts:
- removed P2: SILNIK1, symbol CONN_01X02
- removed P3: SILNIK2, symbol CONN_01X02
- removed U10: L293D, symbol L293D
- added C15, C17, C19, C21: 10uF, symbol CP_Small
- added C16, C18, C20, C22: 0.1uF, symbol C_Small
- added P6: SILNIK1, symbol CONN_01X02
- added P7: SILNIK2, symbol CONN_01X02
- added R11: 100 Ohm, symbol R_Small
- added U11, U12: TB6612, symbol TB6612
- C1, C2, C3, C4: value C_Small -> 1 uF
- C5, C6, C7, C8: value 100uF -> 10uF
- D1: value LED -> DC
- P1: value CONN_01X02 -> bateria 7.4 V
- R1, R2, R3, R4: value R_Small -> 1 Ohm
- gave numbers to parts that had none: 2
Connections:
- net +3V3: now also C15.1, C16.1, C17.1, C18.1, U11.19 (STBY), U11.20 (VCC), U12.19 (STBY), U12.20 (VCC)
- net GND: now also C15.2, C16.2, C17.2, C18.2, C19.2, C20.1, C21.2, C22.1, U11.10 (PGND2), U11.18 (GND), U11.3 (PGND1), U11.4 (PGND1), U11.9 (PGND2), U12.10 (PGND2), U12.18 (GND), U12.3 (PGND1), U12.4 (PGND1), U12.9 (PGND2)
- net VCC: now also P1.1 (P1), SW1.2, C19.1, C20.2, C21.1, C22.2, U11.13 (VM2), U11.14 (VM3), U11.24 (VM1), U12.13 (VM2), U12.14 (VM3), U12.24 (VM1)
- net at U9.40 (PB4/I2S1_MCK/SPI1_MISO/TIM3_CH1/TSC_G5_IO2): now also R11.2; no longer DB1.2 (A)
- net PWD1 renamed 1/ABIN1
- net 1/ABIN1: now also U11.17 (BIN1), U11.21 (AIN1)
- net PWD2 renamed 2/ABIN1
- net 2/ABIN1: now also U12.17 (BIN1), U12.21 (AIN1)
- net WEJSCIE1 renamed 1/PWMAB
- net 1/PWMAB: now also U11.15 (PWMB), U11.23 (PWMA)
- net WEJSCIE2 renamed 1/ABIN2
- net 1/ABIN2: now also U11.16 (BIN2), U11.22 (AIN2)
- net WEJSCIE3 renamed 2/PWMAB
- net 2/PWMAB: now also U12.15 (PWMB), U12.23 (PWMA)
- net WEJSCIE4 renamed 2/ABIN2
- net 2/ABIN2: now also U12.16 (BIN2), U12.22 (AIN2)
- new net: DB1.2 (A), R11.1
- new net: P6.1 (P1), U11.1 (AO1), U11.11 (BO1), U11.12 (BO1), U11.2 (AO1)
- new net: P6.2 (P2), U11.5 (AO2), U11.6 (AO2), U11.7 (BO2), U11.8 (BO2)
- new net: P7.1 (P1), U12.1 (AO1), U12.11 (BO1), U12.12 (BO1), U12.2 (AO1)
- new net: P7.2 (P2), U12.5 (AO2), U12.6 (AO2), U12.7 (BO2), U12.8 (BO2)
Other:
- moved on the sheet: C6, C8, D1, R10, R6, R7, R8, R9, U7, U8

Commit message: Chyba Skończony schemat
Parts:
- removed C19: 10uF, symbol CP_Small
- removed C20: 0.1uF, symbol C_Small
- removed P6: SILNIK1, symbol CONN_01X02
- removed U11: TB6612, symbol TB6612
- added C19: 0.1uF, symbol C_Small
- added C20: 10uF, symbol CP_Small
- added P2: HC-06 (BT), symbol CONN_01X04
- added P3: SILNIK1, symbol CONN_01X02
- added R12: 100 Ohm, symbol R_Small
- added U10: TB6612, symbol TB6612
- D1: value DC -> LED0
- DB1: value LED -> LED1
- DN1: value LED -> LED2
- SP1: value SPEAKER -> HCM1201X (BUZZER)
Connections:
- net 1/ABIN1 is gone; now on net SHARP1: U9.10 (ADC_IN0/COMP1_INM/COMP1_OUT/RTC_TAMP2/SYS_WKUP1/TIM2_CH1/TIM2_ETR/TSC_G1_IO1/USART2_CTS/PA0)
- net 1/ABIN2 is gone; now on net SHARP2: U9.12 (ADC_IN2/COMP2_INM/COMP2_OUT/TIM15_CH1/TIM2_CH3/TSC_G1_IO3/USART2_TX/PA2)
- net 1/PWMAB is gone; now on net KTIR1: U9.11 (ADC_IN1/COMP1_INP/TIM2_CH2/TSC_G1_IO2/USART2_DE/USART2_RTS/PA1)
- net +3V3: now also C10.1, U10.19 (STBY), U10.20 (VCC); no longer C10.2
- net +5V: now also P2.4 (P4)
- net GND: now also C10.2, P1.1 (P1), P4.2 (P2), C19.1, C20.2, P2.3 (P3), U10.10 (PGND2), U10.18 (GND), U10.3 (PGND1), U10.4 (PGND1), U10.9 (PGND2); no longer C10.1, P1.2 (P2), P4.1 (P1), U9.42 (PB6/I2C1_SCL/TIM16_CH1N/TSC_G5_IO3/USART1_TX), U9.43 (PB7/I2C1_SDA/TIM17_CH1N/TSC_G5_IO4/USART1_RX)
- net KTIR1: no longer U9.30 (DAC1_EXTI9/TIM15_BKIN/TIM1_CH2/TSC_G4_IO1/USART1_TX/PA9)
- net KTIR2: now also U9.14 (ADC_IN4/COMP1_INM/COMP2_INM/DAC1_OUT1/I2S1_WS/SPI1_NSS/TIM14_CH1/TSC_G2_IO1/USART2_CK/PA4); no longer U9.33 (COMP2_OUT/TIM1_ETR/TSC_G4_IO4/USART1_DE/USART1_RTS/PA12)
- net SHARP1: no longer U9.29 (RCC_MCO/TIM1_CH1/USART1_CK/PA8)
- net SHARP2: no longer U9.31 (TIM17_BKIN/TIM1_CH3/TSC_G4_IO2/USART1_RX/PA10)
- net SHARP3: now also U9.13 (ADC_IN3/COMP2_INP/TIM15_CH2/TIM2_CH4/TSC_G1_IO4/USART2_RX/PA3); no longer U9.32 (COMP1_OUT/TIM1_CH4/TSC_G4_IO3/USART1_CTS/PA11)
- net SHARP4: now also U9.15 (ADC_IN5/CEC/COMP1_INM/COMP2_INM/I2S1_CK/SPI1_SCK/TIM2_CH1/TIM2_ETR/TSC_G2_IO2/PA5); no longer U9.34 (IR_OUT/SYS_SWDIO/PA13)
- net VCC: now also C5.1, SW1.1, U1.1 (VI), C19.2, C20.1, U10.13 (VM2), U10.14 (VM3), U10.24 (VM1); no longer P1.1 (P1), SW1.2
- net MOD_START: now reaches U9.19 (PB1/ADC_IN9/TIM14_CH1/TIM1_CH3N/TIM3_CH4/TSC_G3_IO3)
- net MOD_START: now also P4.1 (P1)
- net BUZZ: now reaches U9.20 (PB2/TSC_G3_IO4)
- net BUZZ: now also R12.1
- net LED2: now reaches U9.21 (PB10/CEC/I2C2_SCL/TIM2_CH3/TSC_SYNC)
- net LED2: now also R5.2; no longer P5.3 (P3)
- net LED1: now reaches U9.22 (PB11/I2C2_SDA/TIM2_CH4/TSC_G6_IO1)
- net LED1: now also R11.2; no longer P5.2 (P2)
- net S1/IN1: now reaches U9.25 (PB12/SPI2_NSS/TIM1_BKIN/TSC_G6_IO2)
- net S1/IN1: now also U10.17 (BIN1), U10.21 (AIN1)
- net S1/IN2: now reaches U9.26 (PB13/SPI2_SCK/TIM1_CH1N/TSC_G6_IO3)
- net S1/IN2: now also U10.16 (BIN2), U10.22 (AIN2)
- net S1/PWM: now reaches U9.27 (PB14/SPI2_MISO/TIM15_CH1/TIM1_CH2N/TSC_G6_IO4)
- net S1/PWM: now also U10.15 (PWMB), U10.23 (PWMA)
- net S2/PWM: now reaches U9.28 (PB15/RTC_REFIN/SPI2_MOSI/TIM15_CH1N/TIM15_CH2/TIM1_CH3N)
- net S2/PWM: now also U12.15 (PWMB), U12.23 (PWMA)
- net PROG2: now reaches U9.37 (SYS_SWCLK/USART2_TX/PA14)
- net PROG2: now also P5.2 (P2)
- net at U9.39 (PB3/I2S1_CK/SPI1_SCK/TIM2_CH2/TSC_G5_IO1): no longer R5.2
- net at U9.40 (PB4/I2S1_MCK/SPI1_MISO/TIM3_CH1/TSC_G5_IO2): no longer R11.2
- net at U9.41 (PB5/I2C1_SMBA/I2S1_SD/SPI1_MOSI/TIM16_BKIN/TIM3_CH2): no longer SP1.2
- net at U9.45 (PB8/CEC/I2C1_SCL/TIM16_CH1/TSC_SYNC): no longer P4.2 (P2)
- net RESET: now reaches C9.2, SW2.2, U9.7 (NRST)
- net 2/ABIN1 renamed S2/IN1
- net S2/IN1: now also U9.30 (DAC1_EXTI9/TIM15_BKIN/TIM1_CH2/TSC_G4_IO1/USART1_TX/PA9); no longer U9.13 (ADC_IN3/COMP2_INP/TIM15_CH2/TIM2_CH4/TSC_G1_IO4/USART2_RX/PA3)
- net 2/ABIN2 renamed S2/IN2
- net S2/IN2: now also U9.31 (TIM17_BKIN/TIM1_CH3/TSC_G4_IO2/USART1_RX/PA10); no longer U9.15 (ADC_IN5/CEC/COMP1_INM/COMP2_INM/I2S1_CK/SPI1_SCK/TIM2_CH1/TIM2_ETR/TSC_G2_IO2/PA5)
- removed net 2/PWMAB: U12.15 (PWMB), U12.23 (PWMA), U9.14 (ADC_IN4/COMP1_INM/COMP2_INM/DAC1_OUT1/I2S1_WS/SPI1_NSS/TIM14_CH1/TSC_G2_IO1/USART2_CK/PA4)
- new net: P1.2 (P2), SW1.2
- new net: R12.2, SP1.2
- new net: P3.1 (P1), U10.1 (AO1), U10.11 (BO1), U10.12 (BO1), U10.2 (AO1)
- new net: P3.2 (P2), U10.5 (AO2), U10.6 (AO2), U10.7 (BO2), U10.8 (BO2)
- new net BT1: P2.2 (P2), U9.42 (PB6/I2C1_SCL/TIM16_CH1N/TSC_G5_IO3/USART1_TX)
- new net BT2: P2.1 (P1), U9.43 (PB7/I2C1_SDA/TIM17_CH1N/TSC_G5_IO4/USART1_RX)
- new net PROG1: P5.3 (P3), U9.34 (IR_OUT/SYS_SWDIO/PA13)
Other:
- note added: "Czujniki \nSHARP i KTIR"
- note added: "Moduły Komunikacyjne"
- note added: "Mostki H \n"
- note added: "Stabilizacja zasilania: \n STM Mostki H"
- note added: "Zasilanie I Dzielniki napięcia"
- note added: "diody LED"
- moved on the sheet: C1, C10, C11, C12, C13, C14, C17, C18, C2, C21, C22, C3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

Commit message: poprawka
Connections:
- net BUZZ: now also R12.2; no longer R12.1
- net GND: now also C1.1, C2.1, C3.1, C4.1; no longer C1.2, C2.2, C3.2, C4.2
- net at U4.5 (REG): now also C3.2; no longer C3.1
- net at U5.5 (REG): now also C4.2; no longer C4.1
- net at U2.5 (REG): now also C1.2; no longer C1.1
- net at U3.5 (REG): now also C2.2; no longer C2.1
- net at SP1.2: now also R12.1; no longer R12.2
Other:
- note added: "Stabilizacja zasilania STM"
- note removed: "Stabilizacja zasilania: \n STM Mostki H"
- moved on the sheet: C1, C10, C11, C12, C13, C14, C15, C16, C17, C18, C19, C2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

Commit message: footprinty zrobione
Parts:
- removed SW1: SWITCH_INV, symbol SWITCH_INV
- added SW1: SPST, Buttons_Switches_ThroughHole:SW_DIP_x1_Slide, symbol SPST
- C1, C13, C2, C3, C4: footprint (none) -> Capacitors_SMD:C_0402
- C10, C11, C12: footprint (none) -> Capacitors_SMD:C_0603
- C14, C16, C18, C19, C22, C9: footprint (none) -> Capacitors_SMD:C_0805
- C15, C17, C20, C21, C5, C6, C7, C8: footprint (none) -> Capacitors_Tantalum_SMD:TantalC_SizeR_EIA-2012
- D1, DB1, DN1: footprint (none) -> LEDs:LED-5MM
- P1, P3, P7: footprint (none) -> Socket_Strips:Socket_Strip_Straight_1x02
- P2, P5: footprint (none) -> Socket_Strips:Socket_Strip_Straight_1x04
- P4: footprint (none) -> Socket_Strips:Socket_Strip_Straight_1x03
- R1, R11, R12, R2, R3, R4, R5, R6: footprint (none) -> Resistors_SMD:R_0805
- R10, R7, R8, R9: footprint (none) -> Resistors_SMD:R_0603
- SP1: footprint (none) -> Buzzers_Beepers:Buzzer_12x9.5RM7.6
- SW2: footprint (none) -> Buttons_Switches_ThroughHole:SW_PUSH_6mm
- U1, U6: footprint (none) -> warsztaty:LM1117_SOT223
- U10, U12: footprint (none) -> warsztaty:TB6612
- U2, U3, U4, U5: footprint (none) -> warsztaty:GP2Y0D340K
- U7, U8: footprint (none) -> warsztaty:KTIR0711S
- U9: footprint LQFP48 -> STM:STM32F051C8T6
Connections:
- net VCC: now also SW1.2
- net at P1.2 (P2): now also SW1.1
- no-connect marks 22 -> 21
Other:
- moved on the sheet: P1

Commit message: plytka_pcb
Connections:
- net KTIR1: now also U9.26 (PB13/SPI2_SCK/TIM1_CH1N/TSC_G6_IO3); no longer U9.11 (ADC_IN1/COMP1_INP/TIM2_CH2/TSC_G1_IO2/USART2_DE/USART2_RTS/PA1)
- net KTIR2: now also U9.29 (RCC_MCO/TIM1_CH1/USART1_CK/PA8); no longer U9.14 (ADC_IN4/COMP1_INM/COMP2_INM/DAC1_OUT1/I2S1_WS/SPI1_NSS/TIM14_CH1/TSC_G2_IO1/USART2_CK/PA4)
- net S1/IN1: now also U9.15 (ADC_IN5/CEC/COMP1_INM/COMP2_INM/I2S1_CK/SPI1_SCK/TIM2_CH1/TIM2_ETR/TSC_G2_IO2/PA5); no longer U9.25 (PB12/SPI2_NSS/TIM1_BKIN/TSC_G6_IO2)
- net S1/IN2: now also U9.14 (ADC_IN4/COMP1_INM/COMP2_INM/DAC1_OUT1/I2S1_WS/SPI1_NSS/TIM14_CH1/TSC_G2_IO1/USART2_CK/PA4); no longer U9.26 (PB13/SPI2_SCK/TIM1_CH1N/TSC_G6_IO3)
- net S1/PWM: now also U9.13 (ADC_IN3/COMP2_INP/TIM15_CH2/TIM2_CH4/TSC_G1_IO4/USART2_RX/PA3); no longer U9.27 (PB14/SPI2_MISO/TIM15_CH1/TIM1_CH2N/TSC_G6_IO4)
- net S2/IN1: now also U9.10 (ADC_IN0/COMP1_INM/COMP1_OUT/RTC_TAMP2/SYS_WKUP1/TIM2_CH1/TIM2_ETR/TSC_G1_IO1/USART2_CTS/PA0); no longer U9.30 (DAC1_EXTI9/TIM15_BKIN/TIM1_CH2/TSC_G4_IO1/USART1_TX/PA9)
- net S2/IN2: now also U9.11 (ADC_IN1/COMP1_INP/TIM2_CH2/TSC_G1_IO2/USART2_DE/USART2_RTS/PA1); no longer U9.31 (TIM17_BKIN/TIM1_CH3/TSC_G4_IO2/USART1_RX/PA10)
- net S2/PWM: now also U9.12 (ADC_IN2/COMP2_INM/COMP2_OUT/TIM15_CH1/TIM2_CH3/TSC_G1_IO3/USART2_TX/PA2); no longer U9.28 (PB15/RTC_REFIN/SPI2_MOSI/TIM15_CH1N/TIM15_CH2/TIM1_CH3N)
- net SHARP1: now also U9.25 (PB12/SPI2_NSS/TIM1_BKIN/TSC_G6_IO2); no longer U9.10 (ADC_IN0/COMP1_INM/COMP1_OUT/RTC_TAMP2/SYS_WKUP1/TIM2_CH1/TIM2_ETR/TSC_G1_IO1/USART2_CTS/PA0)
- net SHARP2: now also U9.27 (PB14/SPI2_MISO/TIM15_CH1/TIM1_CH2N/TSC_G6_IO4); no longer U9.12 (ADC_IN2/COMP2_INM/COMP2_OUT/TIM15_CH1/TIM2_CH3/TSC_G1_IO3/USART2_TX/PA2)
- net SHARP3: now also U9.28 (PB15/RTC_REFIN/SPI2_MOSI/TIM15_CH1N/TIM15_CH2/TIM1_CH3N); no longer U9.13 (ADC_IN3/COMP2_INP/TIM15_CH2/TIM2_CH4/TSC_G1_IO4/USART2_RX/PA3)
- net SHARP4: now also U9.30 (DAC1_EXTI9/TIM15_BKIN/TIM1_CH2/TSC_G4_IO1/USART1_TX/PA9); no longer U9.15 (ADC_IN5/CEC/COMP1_INM/COMP2_INM/I2S1_CK/SPI1_SCK/TIM2_CH1/TIM2_ETR/TSC_G2_IO2/PA5)
Changed lines of the file:
@@
 	1    0    0    -1
 $EndComp
-Text GLabel 10940 5120 2    60   Input ~ 0
+Text GLabel 4340 6320 0    60   Input ~ 0
 SHARP1
-Text GLabel 10940 5220 2    60   Input ~ 0
+Text GLabel 4340 6420 0    60   Input ~ 0
 KTIR1
-Text GLabel 10940 5320 2    60   Input ~ 0
+Text GLabel 4340 6520 0    60   Input ~ 0
 SHARP2
-Text GLabel 10940 5420 2    60   Input ~ 0
+Text GLabel 4340 6620 0    60   Input ~ 0
 SHARP3
-Text GLabel 10940 5520 2    60   Input ~ 0
+Text GLabel 10940 5920 2    60   Input ~ 0
 KTIR2
-Text GLabel 10940 5620 2    60   Input ~ 0
+Text GLabel 10940 6020 2    60   Input ~ 0
 SHARP4
 Text GLabel 1640 4200 0    60   Input ~ 0
@@
 	-1   0    0    1
 $EndComp
-Text GLabel 4340 6320 0    60   Input ~ 0
+Text GLabel 10940 5620 2    60   Input ~ 0
 S1/IN1
-Text GLabel 4340 6420 0    60   Input ~ 0
+Text GLabel 10940 5520 2    60   Input ~ 0
 S1/IN2
-Text GLabel 10940 6120 2    60   Input ~ 0
+Text GLabel 10940 5220 2    60   Input ~ 0
 S2/IN2
-Text GLabel 10940 6020 2    60   Input ~ 0
+Text GLabel 10940 5120 2    60   Input ~ 0
 S2/IN1
-Text GLabel 4340 6520 0    60   Input ~ 0
+Text GLabel 10940 5420 2    60   Input ~ 0
 S1/PWM
-Text GLabel 4340 6620 0    60   Input ~ 0
+Text GLabel 10940 5320 2    60   Input ~ 0
 S2/PWM
 Text GLabel 4340 6220 0    60   Input ~ 0
@@
 NoConn ~ 4340 5520
 NoConn ~ 4340 5620
-NoConn ~ 10940 5920
 NoConn ~ 10940 6320
 NoConn ~ 10940 6220
@@
 	1    0    0    -1
 $EndComp
+NoConn ~ 10940 6120
 $EndSCHEMATC

Commit message: 2 wersja plytek
Parts:
- C1, C13, C2, C3, C4: footprint Capacitors_SMD:C_0402 -> Capacitors_SMD:C_0805_HandSoldering
- C10, C11, C12: footprint Capacitors_SMD:C_0603 -> Capacitors_SMD:C_0603_HandSoldering
- C14, C16, C18, C19, C22, C9: footprint Capacitors_SMD:C_0805 -> Capacitors_SMD:C_0805_HandSoldering
- C15, C17, C20, C21, C5, C6, C7, C8: footprint Capacitors_Tantalum_SMD:TantalC_SizeR_EIA-2012 -> Capacitors_Tantalum_SMD:Tantalum_Case-A_EIA-3216-18_Hand
- R1, R11, R12, R2, R3, R4, R5, R6: footprint Resistors_SMD:R_0805 -> Resistors_SMD:R_0805_HandSoldering
- R10, R7, R8, R9: footprint Resistors_SMD:R_0603 -> Resistors_SMD:R_0603_HandSoldering
Changed lines of the file:
@@
 F 0 "R6" H 1180 2050 50  0000 L CNN
 F 1 "100 Ohm" H 1180 1990 50  0000 L CNN
-F 2 "Resistors_SMD:R_0805" H 1150 2030 50  0001 C CNN
+F 2 "Resistors_SMD:R_0805_HandSoldering" H 1150 2030 50  0001 C CNN
 F 3 "" H 1150 2030 50  0000 C CNN
 	1    1150 2030
@@
 F 0 "C6" H 4540 1160 50  0000 L CNN
 F 1 "10uF" H 4540 1010 50  0000 L CNN
-F 2 "Capacitors_Tantalum_SMD:TantalC_SizeR_EIA-2012" H 4530 1090 50  0001 C CNN
+F 2 "Capacitors_Tantalum_SMD:Tantalum_Case-A_EIA-3216-18_Hand" H 4530 1090 50  0001 C CNN
 F 3 "" H 4530 1090 50  0000 C CNN
 	1    4530 1090
@@
 F 0 "C5" H 3430 1160 50  0000 L CNN
 F 1 "10uF" H 3430 1010 50  0000 L CNN
-F 2 "Capacitors_Tantalum_SMD:TantalC_SizeR_EIA-2012" H 3420 1090 50  0001 C CNN
+F 2 "Capacitors_Tantalum_SMD:Tantalum_Case-A_EIA-3216-18_Hand" H 3420 1090 50  0001 C CNN
 F 3 "" H 3420 1090 50  0000 C CNN
 	1    3420 1090
@@
 F 0 "R3" H 1440 4020 50  0000 L CNN
 F 1 "1 Ohm" H 1440 3960 50  0000 L CNN
-F 2 "Resistors_SMD:R_0805" H 1410 4000 50  0001 C CNN
+F 2 "Resistors_SMD:R_0805_HandSoldering" H 1410 4000 50  0001 C CNN
 F 3 "" H 1410 4000 50  0000 C CNN
 	1    1410 4000
@@
 F 0 "C3" H 1490 4570 50  0000 L CNN
 F 1 "1 uF" H 1490 4420 50  0000 L CNN
-F 2 "Capacitors_SMD:C_0402" H 1480 4500 50  0001 C CNN
+F 2 "Capacitors_SMD:C_0805_HandSoldering" H 1480 4500 50  0001 C CNN
 F 3 "" H 1480 4500 50  0000 C CNN
 	1    1480 4500
@@
 F 0 "R8" H 2180 8720 50  0000 L CNN
 F 1 "10 kOhm" H 2180 8660 50  0000 L CNN
-F 2 "Resistors_SMD:R_0603" H 2150 8700 50  0001 C CNN
+F 2 "Resistors_SMD:R_0603_HandSoldering" H 2150 8700 50  0001 C CNN
 F 3 "" H 2150 8700 50  0000 C CNN
 	1    2150 8700
@@
 F 0 "R7" H 1190 8630 50  0000 L CNN
 F 1 "220 Ohm" H 1190 8570 50  0000 L CNN
-F 2 "Resistors_SMD:R_0603" H 1160 8610 50  0001 C CNN
+F 2 "Resistors_SMD:R_0603_HandSoldering" H 1160 8610 50  0001 C CNN
 F 3 "" H 1160 8610 50  0000 C CNN
 	1    1160 8610
@@
 F 0 "C8" H 6070 1160 50  0000 L CNN
 F 1 "10uF" H 6070 1010 50  0000 L CNN
-F 2 "Capacitors_Tantalum_SMD:TantalC_SizeR_EIA-2012" H 6060 1090 50  0001 C CNN
+F 2 "Capacitors_Tantalum_SMD:Tantalum_Case-A_EIA-3216-18_Hand" H 6060 1090 50  0001 C CNN
 F 3 "" H 6060 1090 50  0000 C CNN
 	1    6060 1090
@@
 F 0 "C7" H 4960 1160 50  0000 L CNN
 F 1 "10uF" H 4960 1010 50  0000 L CNN
-F 2 "Capacitors_Tantalum_SMD:TantalC_SizeR_EIA-2012" H 4950 1090 50  0001 C CNN
+F 2 "Capacitors_Tantalum_SMD:Tantalum_Case-A_EIA-3216-18_Hand" H 4950 1090 50  0001 C CNN
 F 3 "" H 4950 1090 50  0000 C CNN
 	1    4950 1090
@@
 F 0 "R4" H 1440 5040 50  0000 L CNN
 F 1 "1 Ohm" H 1440 4980 50  0000 L CNN
-F 2 "Resistors_SMD:R_0805" H 1410 5020 50  0001 C CNN
+F 2 "Resistors_SMD:R_0805_HandSoldering" H 1410 5020 50  0001 C CNN
 F 3 "" H 1410 5020 50  0000 C CNN
 	1    1410 5020
@@
 F 0 "C4" H 1490 5590 50  0000 L CNN
 F 1 "1 uF" H 1490 5440 50  0000 L CNN
-F 2 "Capacitors_SMD:C_0402" H 1480 5520 50  0001 C CNN
+F 2 "Capacitors_SMD:C_0805_HandSoldering" H 1480 5520 50  0001 C CNN
 F 3 "" H 1480 5520 50  0000 C CNN
 	1    1480 5520
@@
 F 0 "C1" H 1480 6670 50  0000 L CNN
 F 1 "1 uF" H 1480 6520 50  0000 L CNN
-F 2 "Capacitors_SMD:C_0402" H 1470 6600 50  0001 C CNN
+F 2 "Capacitors_SMD:C_0805_HandSoldering" H 1470 6600 50  0001 C CNN
 F 3 "" H 1470 6600 50  0000 C CNN
 	1    1470 6600
@@
 F 0 "R2" H 1430 7280 50  0000 L CNN
 F 1 "1 Ohm" H 1430 7220 50  0000 L CNN
-F 2 "Resistors_SMD:R_0805" H 1400 7260 50  0001 C CNN
+F 2 "Resistors_SMD:R_0805_HandSoldering" H 1400 7260 50  0001 C CNN
 F 3 "" H 1400 7260 50  0000 C CNN
 	1    1400 7260
@@
 F 0 "C2" H 1480 7830 50  0000 L CNN
 F 1 "1 uF" H 1480 7680 50  0000 L CNN
-F 2 "Capacitors_SMD:C_0402" H 1470 7760 50  0001 C CNN
+F 2 "Capacitors_SMD:C_0805_HandSoldering" H 1470 7760 50  0001 C CNN
 F 3 "" H 1470 7760 50  0000 C CNN
 	1    1470 7760
@@
 F 0 "R10" H 2180 10140 50  0000 L CNN
 F 1 "10 kOhm" H 2180 10080 50  0000 L CNN
-F 2 "Resistors_SMD:R_0603" H 2150 10120 50  0001 C CNN
+F 2 "Resistors_SMD:R_0603_HandSoldering" H 2150 10120 50  0001 C CNN
 F 3 "" H 2150 10120 50  0000 C CNN
 	1    2150 10120
@@
 F 0 "R9" H 1190 10050 50  0000 L CNN
 F 1 "220 Ohm" H 1190 9990 50  0000 L CNN
-F 2 "Resistors_SMD:R_0603" H 1160 10030 50  0001 C CNN
+F 2 "Resistors_SMD:R_0603_HandSoldering" H 1160 10030 50  0001 C CNN
 F 3 "" H 1160 10030 50  0000 C CNN
 	1    1160 10030
@@
 F 0 "C14" H 8190 1860 50  0000 L CNN
 F 1 "10nF" H 8190 1710 50  0000 L CNN
-F 2 "Capacitors_SMD:C_0805" H 8180 1790 50  0001 C CNN
+F 2 "Capacitors_SMD:C_0805_HandSoldering" H 8180 1790 50  0001 C CNN
 F 3 "" H 8180 1790 50  0000 C CNN
 	1    8180 1790
@@
 F 0 "C12" H 7640 1860 50  0000 L CNN
 F 1 "4.7uF" H 7640 1710 50  0000 L CNN
-F 2 "Capacitors_SMD:C_0603" H 7630 1790 50  0001 C CNN
+F 2 "Capacitors_SMD:C_0603_HandSoldering" H 7630 1790 50  0001 C CNN
 F 3 "" H 7630 1790 50  0000 C CNN
 	1    7630 1790
@@
 F 0 "C11" H 7930 1860 50  0000 L CNN
 F 1 "100nF" H 7930 1710 50  0000 L CNN
-F 2 "Capacitors_SMD:C_0603" H 7920 1790 50  0001 C CNN
+F 2 "Capacitors_SMD:C_0603_HandSoldering" H 7920 1790 50  0001 C CNN
 F 3 "" H 7920 1790 50  0000 C CNN
 	1    7920 1790
@@
 F 0 "C10" H 7320 1860 50  0000 L CNN
 F 1 "100nF" H 7320 1710 50  0000 L CNN
-F 2 "Capacitors_SMD:C_0603" H 7310 1790 50  0001 C CNN
+F 2 "Capacitors_SMD:C_0603_HandSoldering" H 7310 1790 50  0001 C CNN
 F 3 "" H 7310 1790 50  0000 C CNN
 	1    7310 1790
@@
 F 0 "C13" H 8420 1860 50  0000 L CNN
 F 1 "1uF" H 8420 1710 50  0000 L CNN
-F 2 "Capacitors_SMD:C_0402" H 8410 1790 50  0001 C CNN
+F 2 "Capacitors_SMD:C_0805_HandSoldering" H 8410 1790 50  0001 C CNN
 F 3 "" H 8410 1790 50  0000 C CNN
 	1    8410 1790
@@
 F 0 "C9" H 9180 9280 50  0000 L CNN
 F 1 "0.1uF" H 9180 9130 50  0000 L CNN
-F 2 "Capacitors_SMD:C_0805" H 9170 9210 50  0001 C CNN
+F 2 "Capacitors_SMD:C_0805_HandSoldering" H 9170 9210 50  0001 C CNN
 F 3 "" H 9170 9210 50  0000 C CNN
 	1    9170 9210
@@
 F 0 "R5" H 1180 2910 50  0000 L CNN
 F 1 "100 Ohm" H 1180 2850 50  0000 L CNN
-F 2 "Resistors_SMD:R_0805" H 1150 2890 50  0001 C CNN
+F 2 "Resistors_SMD:R_0805_HandSoldering" H 1150 2890 50  0001 C CNN
 F 3 "" H 1150 2890 50  0000 C CNN
 	1    1150 2890
@@
 F 0 "C18" H 9850 1850 50  0000 L CNN
 F 1 "0.1uF" H 9850 1700 50  0000 L CNN
-F 2 "Capacitors_SMD:C_0805" H 9840 1780 50  0001 C CNN
+F 2 "Capacitors_SMD:C_0805_HandSoldering" H 9840 1780 50  0001 C CNN
 F 3 "" H 9840 1780 50  0000 C CNN
 	1    9840 1780
@@
 F 0 "C22" H 10270 1850 50  0000 L CNN
 F 1 "0.1uF" H 10270 1700 50  0000 L CNN
-F 2 "Capacitors_SMD:C_0805" H 10260 1780 50  0001 C CNN
+F 2 "Capacitors_SMD:C_0805_HandSoldering" H 10260 1780 50  0001 C CNN
 F 3 "" H 10260 1780 50  0000 C CNN
 	1    10260 1780
@@
 F 0 "C17" H 9620 1850 50  0000 L CNN
 F 1 "10uF" H 9620 1700 50  0000 L CNN
-F 2 "Capacitors_Tantalum_SMD:TantalC_SizeR_EIA-2012" H 9610 1780 50  0001 C CNN
+F 2 "Capacitors_Tantalum_SMD:Tantalum_Case-A_EIA-3216-18_Hand" H 9610 1780 50  0001 C CNN
 F 3 "" H 9610 1780 50  0000 C CNN
 	1    9610 1780
@@
 F 0 "C21" H 10500 1850 50  0000 L CNN
 F 1 "10uF" H 10500 1700 50  0000 L CNN
-F 2 "Capacitors_Tantalum_SMD:TantalC_SizeR_EIA-2012" H 10490 1780 50  0001 C CNN
+F 2 "Capacitors_Tantalum_SMD:Tantalum_Case-A_EIA-3216-18_Hand" H 10490 1780 50  0001 C CNN
 F 3 "" H 10490 1780 50  0000 C CNN
 	1    10490 1780
@@
 F 0 "R11" H 1190 2460 50  0000 L CNN
 F 1 "100 Ohm" H 1190 2400 50  0000 L CNN
-F 2 "Resistors_SMD:R_0805" H 1160 2440 50  0001 C CNN
+F 2 "Resistors_SMD:R_0805_HandSoldering" H 1160 2440 50  0001 C CNN
 F 3 "" H 1160 2440 50  0000 C CNN
 	1    1160 2440
@@
 F 0 "C16" H 11320 1850 50  0000 L CNN
 F 1 "0.1uF" H 11320 1700 50  0000 L CNN
-F 2 "Capacitors_SMD:C_0805" H 11310 1780 50  0001 C CNN
+F 2 "Capacitors_SMD:C_0805_HandSoldering" H 11310 1780 50  0001 C CNN
 F 3 "" H 11310 1780 50  0000 C CNN
 	1    11310 1780
@@
 F 0 "C19" H 11740 1850 50  0000 L CNN
 F 1 "0.1uF" H 11740 1700 50  0000 L CNN
-F 2 "Capacitors_SMD:C_0805" H 11730 1780 50  0001 C CNN
+F 2 "Capacitors_SMD:C_0805_HandSoldering" H 11730 1780 50  0001 C CNN
 F 3 "" H 11730 1780 50  0000 C CNN
 	1    11730 1780
@@
 F 0 "C15" H 11090 1850 50  0000 L CNN
 F 1 "10uF" H 11090 1700 50  0000 L CNN
-F 2 "Capacitors_Tantalum_SMD:TantalC_SizeR_EIA-2012" H 11080 1780 50  0001 C CNN
+F 2 "Capacitors_Tantalum_SMD:Tantalum_Case-A_EIA-3216-18_Hand" H 11080 1780 50  0001 C CNN
 F 3 "" H 11080 1780 50  0000 C CNN
 	1    11080 1780
@@
 F 0 "C20" H 11970 1850 50  0000 L CNN
 F 1 "10uF" H 11970 1700 50  0000 L CNN
-F 2 "Capacitors_Tantalum_SMD:TantalC_SizeR_EIA-2012" H 11960 1780 50  0001 C CNN
+F 2 "Capacitors_Tantalum_SMD:Tantalum_Case-A_EIA-3216-18_Hand" H 11960 1780 50  0001 C CNN
 F 3 "" H 11960 1780 50  0000 C CNN
 	1    11960 1780
@@
 F 0 "R12" H 6670 8780 50  0000 L CNN
 F 1 "100 Ohm" H 6670 8720 50  0000 L CNN
-F 2 "Resistors_SMD:R_0805" H 6640 8760 50  0001 C CNN
+F 2 "Resistors_SMD:R_0805_HandSoldering" H 6640 8760 50  0001 C CNN
 F 3 "" H 6640 8760 50  0000 C CNN
 	1    6640 8760
@@
 F 0 "R1" H 1430 6120 50  0000 L CNN
 F 1 "1 Ohm" H 1430 6060 50  0000 L CNN
-F 2 "Resistors_SMD:R_0805" H 1400 6100 50  0001 C CNN
+F 2 "Resistors_SMD:R_0805_HandSoldering" H 1400 6100 50  0001 C CNN
 F 3 "" H 1400 6100 50  0000 C CNN
 	1    1400 6100
